Commit message: organizing urdf using xacro

File: course2_ws/src/my_robot_description/urdf/robot_representation.xacro (robot description, xacro)
@@ -1,23 +1,11 @@
 <?xml version="1.0"?>
-<robot name="udemy_robot">
-    <material name="blue">
-        <color rgba="0 0 1 1"/>
-    </material>
-    <material name="red">
-        <color rgba="1 0 0 1"/>
-    </material>
-    <material name="green">
-        <color rgba="0 1 0 1"/>
-    </material>
-    <material name="gray">
-        <color rgba="0.5 0.5 0.5 1"/>
-    </material>
+<robot xmlns:xacro="http://www.ros.org/wiki/xacro">
     <link name="base_link"/>
     <link name="body">
         <visual>
             <geometry>
-                <box size="0.6 0.4 0.2"/>
+                <box size="${body_length} ${body_width} ${body_height}"/>
             </geometry>
-            <origin xyz="0 0 0.1" rpy="0 0 0"/>
+            <origin xyz="0 0 ${body_height/2.0}" rpy="0 0 0"/>
             <material name="blue"/>
         </visual>
@@ -26,7 +14,7 @@
         <visual>
             <geometry>
-                <cylinder radius="0.1" length="0.05"/>
+                <cylinder radius="${wheel_radius}" length="${wheel_thickness}"/>
             </geometry>
-            <origin xyz="0 -0.025 0" rpy="1.57 0 0"/>
+            <origin xyz="0 ${-wheel_thickness/2.0} 0" rpy="${pi/2.0} 0 0"/>
             <material name="gray"/>
         </visual>
@@ -35,7 +23,7 @@
         <visual>
             <geometry>
-                <cylinder radius="0.1" length="0.05"/>
+                <cylinder radius="${wheel_radius}" length="${wheel_thickness}"/>
             </geometry>
-            <origin xyz="0 0.025 0" rpy="-1.57 0 0"/>
+            <origin xyz="0 ${wheel_thickness/2.0} 0" rpy="${-pi/2.0} 0 0"/>
             <material name="gray"/>
         </visual>
@@ -44,5 +32,5 @@
         <visual>
             <geometry>
-                <sphere radius="0.05"/>
+                <sphere radius="${caster_radius}"/>
             </geometry>
             <origin xyz="0 0 0" rpy="0 0 0"/>
@@ -50,13 +38,13 @@
         </visual>
     </link>
-    <joint name="base_body_to_base" type="fixed">
+    <joint name="base_link_to_body" type="fixed">
         <parent link="base_link"/>
         <child link="body"/>
-        <origin xyz="0 0 0.1" rpy="0 0 0"/>
+        <origin xyz="0 0 ${body_height/2.0}" rpy="0 0 0"/>
     </joint>
     <joint name="left_wheel_joint" type="continuous">
         <parent link="body"/>
         <child link="left_wheel"/>
-        <origin xyz="0.15 -0.2 0" rpy="0 0 0"/>
+        <origin xyz="${body_length/4.0} ${-body_width/2.0} 0" rpy="0 0 0"/>
         <axis xyz="0 1 0"/>
     </joint>
@@ -64,5 +52,5 @@
         <parent link="body"/>
         <child link="right_wheel"/>
-        <origin xyz="0.15 0.2 0" rpy="0 0 0"/>
+        <origin xyz="${body_length/4.0} ${body_width/2.0} 0" rpy="0 0 0"/>
         <axis xyz="0 1 0"/>
     </joint>
@@ -70,5 +58,5 @@
         <parent link="body"/>
         <child link="caster_wheel"/>
-        <origin xyz="-0.2 0 -0.05" rpy="0 0 0"/>
+        <origin xyz="${-body_length/3.0} 0 ${-caster_radius}" rpy="0 0 0"/>
         <!-- <axis xyz="0 1 0"/> -->
     </joint>
