Commit message: urdf_inertial_&_collision_tags

File: course2_ws/src/my_robot_description/urdf/common_properties.xacro (robot description, xacro)
@@ -13,3 +13,32 @@
         <color rgba="0.5 0.5 0.5 1"/>
     </material>
+    <!--http://wiki.ros.org/urdf/Tutorials/Adding%20Physical%20and%20Collision%20Properties%20to%20a%20URDF%20Model-->
+    <!--https://en.wikipedia.org/wiki/List_of_moments_of_inertia-->
+    <xacro:macro name="box_inertia" params="m l w h xyz rpy">
+        <inertial>
+            <origin xyz="${xyz}" rpy="${rpy}"/>
+            <mass value="${m}"/>
+            <inertia ixx="${(m/12) * (h*h + l*l)}" ixy="0" ixz="0"
+                     iyy="${(m/12) * (w*w + h*h)}" iyz="0"
+                     izz="${(m/12) * (w*w + l*l)}"/>
+        </inertial>
+    </xacro:macro>
+    <xacro:macro name="wheel_inertia" params="m r h xyz rpy">
+        <inertial>
+            <origin xyz="${xyz}" rpy="${rpy}"/>
+            <mass value="${m}"/>
+            <inertia ixx="${(m/12) * (3*r*r + h*h)}" ixy="0" ixz="0"
+                     iyy="${(m/12) * (3*r*r + h*h)}" iyz="0"
+                     izz="${(m/2) * (r*r)}"/>
+        </inertial>
+    </xacro:macro>
+    <xacro:macro name="caster_inertia" params="m r xyz rpy">
+        <inertial>
+            <origin xyz="${xyz}" rpy="${rpy}"/>
+            <mass value="${m}"/>
+            <inertia ixx="${(2/5) * m * (r*r)}" ixy="0" ixz="0"
+                     iyy="${(2/5) * m * (r*r)}" iyz="0"
+                     izz="${(2/5) * m * (r*r)}"/>
+        </inertial>
+    </xacro:macro>
 </robot>

File: course2_ws/src/my_robot_description/urdf/robot_properties.xacro (robot description, xacro)
@@ -7,3 +7,6 @@
     <xacro:property name="wheel_thickness" value="0.05"/>
     <xacro:property name="caster_radius" value="0.05"/>
+    <xacro:property name="body_mass" value="5.0"/>
+    <xacro:property name="wheel_mass" value="1.0"/>
+    <xacro:property name="caster_mass" value="0.5"/>
 </robot>

File: course2_ws/src/my_robot_description/urdf/robot_representation.xacro (robot description, xacro)
@@ -10,4 +10,12 @@
             <material name="blue"/>
         </visual>
+        <collision>
+            <geometry>
+                <box size="${body_length} ${body_width} ${body_height}"/>
+            </geometry>
+            <origin xyz="0 0 ${body_height/2.0}" rpy="0 0 0"/>
+        </collision>
+        <xacro:box_inertia m="${body_mass}" l="${body_length}" w="${body_width}" h="${body_height}"
+                           xyz="0 0 ${body_height/2.0}" rpy="0 0 0"/>
     </link>
     <link name="left_wheel">
@@ -19,4 +27,12 @@
             <material name="gray"/>
         </visual>
+        <collision>
+            <geometry>
+                <cylinder radius="${wheel_radius}" length="${wheel_thickness}"/>
+            </geometry>
+            <origin xyz="0 ${-wheel_thickness/2.0} 0" rpy="${pi/2.0} 0 0"/>
+        </collision>
+        <xacro:wheel_inertia m="${wheel_mass}" r="${wheel_radius}" h="${wheel_thickness}"
+                             xyz="0 ${-wheel_thickness/2.0} 0" rpy="${pi/2.0} 0 0"/>
     </link>
     <link name="right_wheel">
@@ -28,4 +44,12 @@
             <material name="gray"/>
         </visual>
+        <collision>
+            <geometry>
+                <cylinder radius="${wheel_radius}" length="${wheel_thickness}"/>
+            </geometry>
+            <origin xyz="0 ${wheel_thickness/2.0} 0" rpy="${-pi/2.0} 0 0"/>
+        </collision>
+        <xacro:wheel_inertia m="${wheel_mass}" r="${wheel_radius}" h="${wheel_thickness}"
+                             xyz="0 ${wheel_thickness/2.0} 0" rpy="${-pi/2.0} 0 0"/>
     </link>
     <link name="caster_wheel">
@@ -37,4 +61,12 @@
             <material name="gray"/>
         </visual>
+        <collision>
+            <geometry>
+                <sphere radius="${caster_radius}"/>
+            </geometry>
+            <origin xyz="0 0 0" rpy="0 0 0"/>
+        </collision>
+        <xacro:caster_inertia m="${caster_mass}" r="${caster_radius}"
+                              xyz="0 0 0" rpy="0 0 0"/>
     </link>
     <joint name="base_link_to_body" type="fixed">
