Commit message: Refactoring and fixes

File: course2_ws/src/udemy_robot_description/urdf/robot_properties.xacro (robot description, xacro)
@@ -1,10 +1,28 @@
 <?xml version="1.0"?>
 <robot xmlns:xacro="http://www.ros.org/wiki/xacro">
+    <!-- Dimensions -->
     <xacro:property name="body_length" value="0.6"/>
     <xacro:property name="body_width" value="0.4"/>
     <xacro:property name="body_height" value="0.2"/>
-    <xacro:property name="wheel_radius" value="${body_height/2.0}"/>
+    <xacro:property name="wheel_radius" value="0.1"/>
     <xacro:property name="wheel_thickness" value="0.05"/>
-    <xacro:property name="caster_radius" value="0.05"/>
+    <xacro:property name="caster_radius" value="${wheel_radius/2.0}"/>
+    <!-- Offsets -->
+    <xacro:property name="body_ground_offset_z"
+                    value="${wheel_radius}"/>
+    <xacro:property name="wheel_joint_offset_x"
+                    value="${-body_length / 4.0}"/>
+    <xacro:property name="left_wheel_joint_offset_y"
+                    value="${-(body_width + wheel_thickness)/ 2.0}"/>
+    <xacro:property name="right_wheel_joint_offset_y"
+                    value="${(body_width + wheel_thickness) / 2.0}"/>
+    <xacro:property name="caster_wheel_joint_offset_x"
+                    value="${body_length / 3.0}"/>
+    <xacro:property name="caster_wheel_joint_offset_z"
+                    value="${-wheel_radius / 2.0}"/>
+    <!-- Diff_drive_configs -->
+    <xacro:property name="wheel_separation"
+                    value="${left_wheel_joint_offset_y + right_wheel_joint_offset_y}"/>
+    <!-- Properties -->
     <xacro:property name="body_mass" value="5.0"/>
     <xacro:property name="wheel_mass" value="1.0"/>

File: course2_ws/src/udemy_robot_description/urdf/robot_representation.xacro (robot description, xacro)
@@ -7,5 +7,5 @@
                 <box size="${body_length} ${body_width} ${body_height}"/>
             </geometry>
-            <origin xyz="0 0 ${body_height/2.0}" rpy="0 0 0"/>
+            <origin xyz="0 0 ${body_height / 2.0}" rpy="0 0 0"/>
             <material name="blue"/>
         </visual>
@@ -14,43 +14,30 @@
                 <box size="${body_length} ${body_width} ${body_height}"/>
             </geometry>
-            <origin xyz="0 0 ${body_height/2.0}" rpy="0 0 0"/>
+            <origin xyz="0 0 ${body_height / 2.0}" rpy="0 0 0"/>
         </collision>
         <xacro:box_inertia m="${body_mass}" l="${body_length}" w="${body_width}" h="${body_height}"
-                           xyz="0 0 ${body_height/2.0}" rpy="0 0 0"/>
+                           xyz="0 0 ${body_height / 2.0}" rpy="0 0 0"/>
     </link>
-    <link name="left_wheel">
-        <visual>
-            <geometry>
-                <cylinder radius="${wheel_radius}" length="${wheel_thickness}"/>
-            </geometry>
-            <origin xyz="0 ${-wheel_thickness/2.0} 0" rpy="${pi/2.0} 0 0"/>
-            <material name="gray"/>
-        </visual>
-        <collision>
-            <geometry>
-                <cylinder radius="${wheel_radius}" length="${wheel_thickness}"/>
-            </geometry>
-            <origin xyz="0 ${-wheel_thickness/2.0} 0" rpy="${pi/2.0} 0 0"/>
-        </collision>
-        <xacro:wheel_inertia m="${wheel_mass}" r="${wheel_radius}" h="${wheel_thickness}"
-                             xyz="0 ${-wheel_thickness/2.0} 0" rpy="${pi/2.0} 0 0"/>
-    </link>
-    <link name="right_wheel">
-        <visual>
-            <geometry>
-                <cylinder radius="${wheel_radius}" length="${wheel_thickness}"/>
-            </geometry>
-            <origin xyz="0 ${wheel_thickness/2.0} 0" rpy="${-pi/2.0} 0 0"/>
-            <material name="gray"/>
-        </visual>
-        <collision>
-            <geometry>
-                <cylinder radius="${wheel_radius}" length="${wheel_thickness}"/>
-            </geometry>
-            <origin xyz="0 ${wheel_thickness/2.0} 0" rpy="${-pi/2.0} 0 0"/>
-        </collision>
-        <xacro:wheel_inertia m="${wheel_mass}" r="${wheel_radius}" h="${wheel_thickness}"
-                             xyz="0 ${wheel_thickness/2.0} 0" rpy="${-pi/2.0} 0 0"/>
-    </link>
+    <xacro:macro name="wheel" params="prefix">
+        <link name="${prefix}_wheel">
+            <visual>
+                <geometry>
+                    <cylinder radius="${wheel_radius}" length="${wheel_thickness}" />
+                </geometry>
+                <origin xyz="0 0 0" rpy="${pi / 2.0} 0 0" />
+                <material name="gray" />
+            </visual>
+            <collision>
+                <geometry>
+                    <sphere radius="${wheel_radius}" />
+                </geometry>
+                <origin xyz="0 0 0" rpy="0 0 0" />
+            </collision>
+            <xacro:wheel_inertia m="${wheel_mass}" r="${wheel_radius}" h="${wheel_thickness}"
+                                    xyz="0 0 0" rpy="${pi / 2.0} 0 0" />
+        </link>
+    </xacro:macro>
+    <xacro:wheel prefix="right" />
+    <xacro:wheel prefix="left" />
     <link name="caster_wheel">
         <visual>
@@ -73,10 +60,10 @@
         <parent link="base_link"/>
         <child link="body"/>
-        <origin xyz="0 0 ${body_height/2.0}" rpy="0 0 0"/>
+        <origin xyz="0 0 ${body_ground_offset_z}" rpy="0 0 0"/>
     </joint>
     <joint name="left_wheel_joint" type="continuous">
         <parent link="body"/>
         <child link="left_wheel"/>
-        <origin xyz="${body_length/4.0} ${-body_width/2.0} 0" rpy="0 0 0"/>
+        <origin xyz="${wheel_joint_offset_x} ${left_wheel_joint_offset_y} 0" rpy="0 0 0"/>
         <axis xyz="0 1 0"/>
     </joint>
@@ -84,5 +71,5 @@
         <parent link="body"/>
         <child link="right_wheel"/>
-        <origin xyz="${body_length/4.0} ${body_width/2.0} 0" rpy="0 0 0"/>
+        <origin xyz="${wheel_joint_offset_x} ${right_wheel_joint_offset_y} 0" rpy="0 0 0"/>
         <axis xyz="0 1 0"/>
     </joint>
@@ -90,5 +77,5 @@
         <parent link="body"/>
         <child link="caster_wheel"/>
-        <origin xyz="${-body_length/3.0} 0 ${-caster_radius}" rpy="0 0 0"/>
+        <origin xyz="${caster_wheel_joint_offset_x} 0 ${caster_wheel_joint_offset_z}" rpy="0 0 0"/>
         <!-- <axis xyz="0 1 0"/> -->
     </joint>

File: course2_ws/src/udemy_robot_description/urdf/udemy_robot_gazebo.xacro (robot description, xacro)
@@ -1,8 +1,8 @@
 <?xml version="1.0"?>
-<robot xmlns:xacro="http://ros.org/wiki/xacro" name="udemy_robot">
-    <gazebo reference="caster_wheel_link">
+<robot xmlns:xacro="http://ros.org/wiki/xacro">
+    <gazebo reference="caster_wheel">
     <!-- friction coefficients -->
-        <mu1 value="0.1" />
-        <mu2 value="0.1" />
+        <mu1 value="0.0" />
+        <mu2 value="0.0" />
     </gazebo>
     <gazebo>
